File: sidedriver/sidedriver_v1.brd (EAGLE design)
At the start: 70 x 72 mm, 21 parts, among them IC2 LD117AD2MTR, X1 I2C, X3 1751248

Commit message: zmieniony ksztalt mainb
Parts:
- removed C1: (no value), rcl:C0603
- removed R1: (no value), rcl:R0603
- removed U$5: STM32F407V, stm32f4:TQFP100
- removed X1: I2C, con-maritex:MICROMATCH-4
- added C7: 100n, rcl:C0603
- added C8, C9: 2.2u, rcl:C0603
- added I2C: (no value), con-maritex:MICROMATCH-4
- added JTAG: (no value), con-maritex:MICROMATCH-8
- added L1: 10uH, con-maritex:L0805
- added R4: 200, rcl:R0603
- added R5, R6: 10K, rcl:R0603
- added UC: STM32F405RGT, stm32f4:TQFP64
- C2: value (none) -> i tu tez
- C3: value (none) -> wartosc, tej
- C5, C6: value (none) -> 16p
- ENKODER, KRANC, TRANS: value I2C -> (none)
- Q1: value (none) -> 8MHz; device wb:CFPX-217 -> wb:12SMX
- moved C6 123.2 mm to (58.4, 5.08), turned to 90 degrees
- moved C5 117.5 mm to (53.3, 5.08), turned to 270 degrees
- moved Q1 109.5 mm to (45.7, 5.08)
Connections:
- net 12V renamed +12V
- net 5V renamed +5V
- removed net 3,3V: C2.1, IC2.2, U$3.7, U$4.7
- removed net N$14: U$3.2
- removed net N$16: U$3.6
- removed net N$7: U$4.2
- removed net N$8: U$4.3
- removed net N$9: U$4.6
- new net !JRST: JTAG.1, UC.56
- new net !RST: JTAG.6, UC.7
- new net +3V3: C2.1, C7.1, IC2.2, JTAG.2, L1.1, R5.2, U$3.7, U$4.7, UC.19, UC.32, UC.48, UC.64
- new net 1-ENA: U$4.2, UC.24
- new net 1-INA: U$4.1, UC.23
- new net 1-PWM: U$4.3, UC.25
- new net JTCK: JTAG.7, R6.2, UC.49
- new net JTDI: JTAG.3, UC.50
- new net JTDO: JTAG.4, UC.55
- new net JTMS: JTAG.5, R5.1, UC.46
- new net N$20: L1.2, UC.13
- new net N$22: R4.1, UC.6
- new net N$23: C8.1, UC.47
- new net N$24: C9.1, UC.31
- new net N$25: I2C.1
- new net N$38: U$3.2, UC.37
- new net N$39: U$3.1, UC.38
- new net SCL: I2C.3, UC.29
- new net SDA: I2C.2, UC.30
- net GND: now also C7.2, C8.2, C9.2, I2C.4, JTAG.8, R6.1, UC.12, UC.18, UC.60, UC.63
- net N$10: now also UC.27
- net N$11: now also UC.26
- net N$13: now also U$3.6, UC.33; no longer U$3.1
- net N$15: now also UC.36
- net N$17: now also UC.34
- net N$18: now also UC.35
- net N$4: now also R4.2
- net N$5: now also Q1.3, UC.5; no longer Q1.2
- net N$6: now also U$4.6, UC.28; no longer U$4.1
Routing:
- net +12V: track 85.2 -> 42.6 mm
- net +3V3: track 0.00 -> 26.6 mm, vias 0 -> 1
- net SCL: track 0.00 -> 24.0 mm
- net SDA: track 0.00 -> 20.5 mm
- net GND: track 272.8 -> 277.5 mm
- net N$29: track 0.00 -> 2.79 mm
- net N$30: track 0.00 -> 2.79 mm
- net N$32: track 0.00 -> 2.54 mm
- net N$28: track 0.00 -> 2.54 mm
- net N$27: track 0.00 -> 2.54 mm
- net N$26: track 0.00 -> 2.54 mm
- net N$33: track 0.00 -> 2.29 mm
- net N$31: track 0.00 -> 2.29 mm

Commit message: 21.11.13 23:39
Parts:
- moved R6 22.8 mm to (28.3, 9.40), turned to 180 degrees
- moved R5 15.7 mm to (25.0, 9.40), turned to 180 degrees
- moved C7 13.5 mm to (54.1, 3.05), turned to 180 degrees
- moved L1 9.35 mm to (54.1, 6.35), turned to 180 degrees
- moved C6 8.87 mm to (49.8, 3.05), turned to 0 degrees
- moved R4 7.22 mm to (48.8, 6.35)
- moved C8 6.71 mm to (54.1, 22.1)
- moved C9 3.31 mm to (55.6, 22.1)
- moved C5 2.84 mm to (50.8, 6.35)
- moved I2C 2.79 mm to (58.2, 38.1)
- moved UC 2.65 mm to (48.3, 15.7)
- moved JTAG 2.54 mm to (30.5, 5.08)
- moved Q1 2.54 mm to (43.2, 5.08)
- moved C2 0.38 mm to (22.5, 3.81)
Routing:
- net +3V3: track 26.6 -> 115.6 mm
- net GND: track 277.5 -> 345.1 mm, vias 0 -> 2
- net N$39: track 0.00 -> 51.3 mm
- net N$6: track 0.00 -> 48.6 mm
- net N$38: track 0.00 -> 48.6 mm
- net N$10: track 0.00 -> 46.9 mm
- net N$15: track 0.00 -> 45.9 mm
- net N$11: track 0.00 -> 45.1 mm
- net 1-PWM: track 0.00 -> 43.4 mm
- net N$18: track 0.00 -> 43.1 mm
- net +12V: track 42.6 -> 85.2 mm
- net JTMS: track 0.00 -> 42.1 mm
- net 1-ENA: track 0.00 -> 41.7 mm
- net N$17: track 0.00 -> 40.4 mm
- net 1-INA: track 0.00 -> 39.9 mm
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
Commit message: 26.11 10:46
Parts:
- removed X3: 1751248, con-phoenix-350:1751248
- added C1: (no value), rcl:C0603
- added C10: i tu tez, rcl:C0603
- moved ENKODER 12.7 mm to (33.0, 38.1)
- moved KRANC 12.7 mm to (45.7, 38.1)
- moved C2 0.25 mm to (22.2, 3.81)
Connections:
- removed net N$2: U$2.6, X3.1
- removed net N$3: U$2.5, X3.2
- new net N$7: UC.45
- new net N$8: UC.44
- net +3V3: now also C10.1, C4.1, KRANC.2, KRANC.3, R2.1, R3.1
- net +5V: no longer C4.1, R2.1, R3.1
- net GND: now also C1.1, C10.2; no longer KRANC.2, KRANC.3
- net MAX: now also UC.40
- net MIN: now also UC.39
- net TOR1: now also UC.41
- net TOR2: now also UC.42
- net TRANS: now also C1.2, UC.43
Routing:
- net +3V3: track 115.6 -> 212.6 mm
- net TRANS: track 0.00 -> 46.5 mm
- net GND: track 345.1 -> 384.6 mm
- net TOR1: track 0.00 -> 26.6 mm
- net TOR2: track 0.00 -> 24.8 mm
- net MAX: track 0.00 -> 20.2 mm
- net MIN: track 0.00 -> 15.6 mm
- net +5V: track 37.3 -> 48.4 mm, vias 0 -> 1
- net N$1: track 0.00 -> 4.49 mm

Commit message: 03-12-13 20:52
Parts:
- removed UC: STM32F405RGT, stm32f4:TQFP64
- added U$1: STM32F405R, stm32f4:TQFP64
- added UART: C-GRID-03-70543, con-molex:70543-03
- moved C3 1.27 mm to (3.81, 14.0)
- moved I2C 1.02 mm to (59.2, 38.1), turned to 90 degrees
- renumbered ENKODER to ENC, TRANS to T-OPT
Connections:
- removed net 1-ENA: U$4.2, UC.24
- removed net 1-INA: U$4.1, UC.23
- removed net 1-PWM: U$4.3, UC.25
- removed net N$10: U$4.5, UC.27
- removed net N$11: U$4.4, UC.26
- removed net N$12: U$4.9
- removed net N$13: U$3.6, UC.33
- removed net N$15: U$3.3, UC.36
- removed net N$17: U$3.5, UC.34
- removed net N$18: U$3.4, UC.35
- removed net N$19: U$3.9
- removed net N$21: U$2.2
- removed net N$25: I2C.1
- removed net N$38: U$3.2, UC.37
- removed net N$39: U$3.1, UC.38
- removed net N$6: U$4.6, UC.28
- removed net N$7: UC.45
- removed net N$8: UC.44
- removed net TOR1: ENC.2, UC.41
- removed net TOR2: ENC.4, UC.42
- new net ENC1: ENC.2, U$1.41
- new net ENC2: ENC.4, U$1.44
- new net LED-PWM: U$1.58, U$2.2
- new net M1-CS: U$1.26, U$4.4
- new net M1-ENA: U$1.24, U$4.2
- new net M1-ENB: U$4.5
- new net M1-INA: U$1.23, U$4.1
- new net M1-INB: U$4.6
- new net M1-PWM: U$1.37, U$4.3
- new net M2-CS: U$1.27, U$3.4
- new net M2-ENA: U$3.2
- new net M2-ENB: U$3.5
- new net M2-INA: U$3.1
- new net M2-INB: U$3.6
- new net M2-PWM: U$1.38, U$3.3
- new net RX: U$1.43, UART.2
- new net TX: U$1.42, UART.3
- net !JRST: now also U$1.56; no longer UC.56
- net !RST: now also U$1.7; no longer UC.7
- net +3V3: now also U$1.19, U$1.32, U$1.48, U$1.64; no longer UC.19, UC.32, UC.48, UC.64
- net +5V: now also I2C.4
- net GND: now also I2C.3, U$1.12, U$1.18, U$1.60, U$1.63, UART.1; no longer I2C.4, UC.12, UC.18, UC.60, UC.63
- net JTCK: now also U$1.49; no longer UC.49
- net JTDI: now also U$1.50; no longer UC.50
- net JTDO: now also U$1.55; no longer UC.55
- net JTMS: now also U$1.46; no longer UC.46
- net MAX: no longer UC.40
- net MIN: no longer UC.39
- net N$20: now also U$1.13; no longer UC.13
- net N$22: now also U$1.6; no longer UC.6
- net N$23: now also U$1.47; no longer UC.47
- net N$24: now also U$1.31; no longer UC.31
- net N$5: now also U$1.5; no longer UC.5
- net SCL: now also I2C.2, U$1.29; no longer I2C.3, UC.29
- net SDA: now also I2C.1, U$1.30; no longer I2C.2, UC.30
- net TRANS: no longer UC.43
Routing:
- net GND: track 384.6 -> 0.00 mm, vias 2 -> 0
- net N$39: track 51.3 -> 0.00 mm
- net N$6: track 48.6 -> 0.00 mm
- net N$38: track 48.6 -> 0.00 mm
- net M2-INA: track 0.00 -> 47.4 mm
- net N$10: track 46.9 -> 0.00 mm
- net N$15: track 45.9 -> 0.00 mm
- net M2-ENA: track 0.00 -> 45.2 mm
- net N$11: track 45.1 -> 0.00 mm
- net 1-PWM: track 43.4 -> 0.00 mm
- net N$18: track 43.1 -> 0.00 mm
- net M1-ENB: track 0.00 -> 42.7 mm
- net 1-ENA: track 41.7 -> 0.00 mm
- net M1-CS: track 0.00 -> 40.4 mm
- net N$17: track 40.4 -> 0.00 mm
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- added copper zone on layer 1, net GND
- added copper zone on layer 16, net GND

Commit message: 11.12.13 18:50
Parts:
- added SV2: (no value), con-lstb:MA07-1
- added U$5: (no value), isfar2-logo:I2-LOGO
- IC2: value LD117AD2MTR -> LT1086CM-3.3
- moved U$1 70.5 mm to (52.0, 15.0), turned to 180 degrees
- moved UART 35.7 mm to (19.2, 21.2), turned to 90 degrees
- moved Q1 22.6 mm to (65.5, 8.50), turned to 270 degrees
- moved L1 16.2 mm to (57.9, 22.1), turned to 0 degrees
- moved R5 16.1 mm to (41.1, 10.1)
- moved C8 15.4 mm to (44.6, 10.0), turned to 180 degrees
- moved R4 14.5 mm to (61.8, 12.8)
- moved C4 14.3 mm to (28.2, 34.8), turned to 90 degrees
- moved C6 13.7 mm to (61.8, 9.60), turned to 270 degrees
- moved R3 13.2 mm to (26.8, 34.8), turned to 90 degrees
- moved R2 12.8 mm to (25.4, 34.8), turned to 90 degrees
- moved R6 12.8 mm to (41.1, 8.80)
- moved C7 11.1 mm to (44.6, 8.80)
- moved C5 11.0 mm to (61.8, 6.20), turned to 90 degrees
- moved C9 7.59 mm to (48.3, 24.1)
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Connections:
- new net G_ADC1: SV2.3, U$1.8
- new net G_ADC2: SV2.4, U$1.9
- new net SRV1: SV2.5, U$1.41
- new net SRV2: SV2.6, U$1.44
- net +12V: now also SV2.7; no longer C3.1, IC2.3
- net +5V: now also C3.1, IC2.3, SV2.1
- net ENC1: now also U$1.37; no longer U$1.41
- net ENC2: now also U$1.38; no longer U$1.44
- net GND: now also SV2.2
- net LED-PWM: now also U$1.40; no longer U$1.58
- net M1-CS: now also U$1.16; no longer U$1.26
- net M1-ENA: now also U$1.11; no longer U$1.24
- net M1-ENB: now also U$1.17
- net M1-INA: now also U$1.10; no longer U$1.23
- net M1-INB: now also U$1.20
- net M1-PWM: now also U$1.15; no longer U$1.37
- net M2-CS: now also U$1.23; no longer U$1.27
- net M2-ENA: now also U$1.27
- net M2-ENB: now also U$1.22
- net M2-INA: now also U$1.28
- net M2-INB: now also U$1.21
- net M2-PWM: now also U$1.26; no longer U$1.38
- net MAX: now also U$1.30
- net MIN: now also U$1.29
- net SCL: now also U$1.61; no longer U$1.29
- net SDA: now also U$1.62; no longer U$1.30
- net TRANS: now also U$1.39
Routing:
- net +5V: track 48.4 -> 133.8 mm
- net G_ADC2: track 0.00 -> 63.7 mm, vias 0 -> 2
- net G_ADC1: track 0.00 -> 62.9 mm, vias 0 -> 2
- net SRV2: track 0.00 -> 60.7 mm, vias 0 -> 2
- net LED-PWM: track 0.00 -> 58.2 mm
- net SRV1: track 0.00 -> 57.1 mm, vias 0 -> 2
- net M2-PWM: track 0.00 -> 49.0 mm
- net M1-INB: track 0.00 -> 47.7 mm
- net M2-CS: track 0.00 -> 45.7 mm
- net M2-ENB: track 0.00 -> 42.8 mm
- net !RST: track 0.00 -> 42.4 mm
- net SCL: track 0.00 -> 42.3 mm, vias 0 -> 1
- net M2-INB: track 0.00 -> 39.9 mm
- net SDA: track 0.00 -> 39.0 mm, vias 0 -> 1
- net M1-ENA: track 0.00 -> 38.7 mm
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Other:
- board text added: "+12V"
- board text added: "+5V"
- board text added: "ADC"
- board text added: "GND"
- board text added: "PWM"
