File: sidedriver/sidedriver_v1.sch (EAGLE design)
At the start: 21 parts, among them IC2 LD117AD2MTR, X1 I2C, X3 1751248

Commit message: zmieniony ksztalt mainb
Parts:
- removed C1: (no value), rcl:C-EUC0603
- removed R1: (no value), rcl:R-EU_R0603
- removed U$5: STM32F407V, stm32f4:STM32F407V
- removed X1: I2C, con-maritex:MICROMATCH-4
- added C7: 100n, rcl:C-EUC0603
- added C8, C9: 2.2u, rcl:C-EUC0603
- added I2C: MICROMATCH-4, con-maritex:MICROMATCH-4
- added JTAG: MICROMATCH-8, con-maritex:MICROMATCH-8
- added L1: 10uH, con-maritex:L
- added R4: 200, rcl:R-EU_R0603
- added R5, R6: 10K, rcl:R-EU_R0603
- added UC: STM32F405RGT, stm32f4:STM32F405R
- C2: value (none) -> i tu tez
- C3: value (none) -> wartosc, tej
- C5, C6: value (none) -> 16p
- ENKODER, KRANC, TRANS: value I2C -> MICROMATCH-4
- Q1: value (none) -> 8MHz; device wb:CRYSTAL -> wb:CRYSTAL12SMX
Connections:
- net 12V renamed +12V
- net 5V renamed +5V
- removed net 3,3V: C2.1, IC2.OUT, U$3.VDD, U$4.VDD
- removed net N$14: U$3.ENA/DIAGA
- removed net N$16: U$3.INB
- removed net N$7: U$4.ENA/DIAGA
- removed net N$8: U$4.PWM
- removed net N$9: U$4.INB
- new net !JRST: JTAG-1.S, UC.PB4/JNTRST(5T)
- new net !RST: JTAG-6.S, UC.NRST
- new net +3V3: C2.1, C7.1, IC2.OUT, JTAG-2.S, L1.1, R5.2, U$3.VDD, U$4.VDD, UC.VDD_1, UC.VDD_2, UC.VDD_3, UC.VDD_4
- new net 1-ENA: U$4.ENA/DIAGA, UC.PC4/ADC12_IN14
- new net 1-INA: U$4.INA, UC.PA7/TIM1_CH1N/ADC12_IN7(FT)
- new net 1-PWM: U$4.PWM, UC.PC5/ADC12_IN15
- new net JTCK: JTAG-7.S, R6.2, UC.PA14/JTCK-SWCLK(5T)
- new net JTDI: JTAG-3.S, UC.PA15/JTDI(5T)
- new net JTDO: JTAG-4.S, UC.PB3/JTDO(5T)
- new net JTMS: JTAG-5.S, R5.1, UC.PA13/JTMS-SWDAT(5T)
- new net N$20: L1.2, UC.VDDA
- new net N$22: R4.1, UC.PH1/OSC_OUT(5T)
- new net N$23: C8.1, UC.VCAP_2
- new net N$24: C9.1, UC.VCAP_1
- new net N$25: I2C-1.S
- new net N$38: U$3.ENA/DIAGA, UC.PC6/TIM3_CH1/TIM_CH1/USART6_TX(5T)
- new net N$39: U$3.INA, UC.PC7/TIM3_CH2/TIM8_CH2/USART6_RX(5T)
- new net SCL: I2C-3.S, UC.PB10/I2C2_SCL(5T)
- new net SDA: I2C-2.S, UC.PB11/I2C2_SDA(5T)
- net GND: now also C7.2, C8.2, C9.2, I2C-4.S, JTAG-8.S, R6.1, UC.BOOT0, UC.VSSA, UC.VSS_1, UC.VSS_2
- net N$10: now also UC.PB1/TIM1_CH3N/ADC12_IN9(5T)
- net N$11: now also UC.PB0/TIM1_CH2N/ADC12_IN8(5T)
- net N$13: now also U$3.INB, UC.PB12(5T); no longer U$3.INA
- net N$15: now also UC.PB15/SPI2_MOSI(5T)
- net N$17: now also UC.PB13/SPI2_SCK(5T)
- net N$18: now also UC.PB14/SPI2_MISO(5T)
- net N$4: now also R4.2
- net N$5: now also UC.PH0/OSC_IN(5T)
- net N$6: now also U$4.INB, UC.PB2/BOOT1(5T); no longer U$4.INA
Other:
- moved on the sheet: C2, C3, C5, C6, IC2, Q1, X2-1, X2-2, X2-3

Commit message: 26.11 10:46
Parts:
- removed X3: 1751248, con-phoenix-350:1751248
- added C1: (no value), rcl:C-EUC0603
- added C10: i tu tez, rcl:C-EUC0603
Connections:
- removed net N$2: U$2.LED-, X3-1.K
- removed net N$3: U$2.LED+, X3-2.K
- new net N$7: UC.PA12/CANTX/USBDP(5T)
- new net N$8: UC.PA11/TIM1_CH4/CANRX/USBDM(5T)
- net +3V3: now also C10.1, C4.1, KRANC-2.S, KRANC-3.S, R2.1, R3.1
- net +5V: no longer C4.1, R2.1, R3.1
- net GND: now also C1.1, C10.2; no longer KRANC-2.S, KRANC-3.S
- net MAX: now also UC.PC9/TIM3_CH4/TIM8_CH4(5T)
- net MIN: now also UC.PC8/TIM3_CH3/TIM8_CH3(5T)
- net TOR1: now also UC.PA8/TIM1_CH1(5T)
- net TOR2: now also UC.PA9/TIM1_CH2/USART1_TX(5T)
- net TRANS: now also C1.2, UC.PA10/TIM1_CH3/USART1_RX(5T)
Changed lines of the file:
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@@
 <part name="C4" library="rcl" deviceset="C-EU" device="C0603"/>
 <part name="ENKODER" library="con-maritex" deviceset="MICROMATCH-4" device="" value=""/>
-<part name="X3" library="con-phoenix-350" deviceset="1751248" device=""/>
 <part name="C5" library="rcl" deviceset="C-EU" device="C0603" value="16p"/>
 <part name="C6" library="rcl" deviceset="C-EU" device="C0603" value="16p"/>
@@
 <part name="L1" library="con-maritex" deviceset="L" device="" value="10uH"/>
 <part name="GND15" library="supply1" deviceset="GND" device=""/>
+<part name="C1" library="rcl" deviceset="C-EU" device="C0603"/>
+<part name="C10" library="rcl" deviceset="C-EU" device="C0603" value="i tu tez"/>
+<part name="GND16" library="supply1" deviceset="GND" device=""/>
 </parts>
 <sheets>
@@
 <instance part="ENKODER" gate="-3" x="-15.24" y="-2.54"/>
 <instance part="ENKODER" gate="-4" x="-15.24" y="-5.08"/>
-<instance part="X3" gate="-1" x="269.24" y="7.62"/>
-<instance part="X3" gate="-2" x="269.24" y="15.24"/>
 <instance part="C5" gate="G$1" x="185.42" y="55.88" rot="R90"/>
 <instance part="C6" gate="G$1" x="185.42" y="45.72" rot="MR270"/>
 <instance part="GND1" gate="1" x="193.04" y="35.56"/>
 <instance part="UC" gate="G$1" x="121.92" y="88.9"/>
-<instance part="+3V1" gate="G$1" x="5.08" y="101.6" rot="R270"/>
+<instance part="+3V1" gate="G$1" x="7.62" y="101.6" rot="R270"/>
 <instance part="+3V2" gate="G$1" x="43.18" y="121.92" rot="R90"/>
 <instance part="C7" gate="G$1" x="50.8" y="109.22"/>
@@
 </instance>
 <instance part="GND15" gate="1" x="205.74" y="93.98"/>
+<instance part="C1" gate="G$1" x="-22.86" y="30.48" smashed="yes" rot="R90">
+<attribute name="NAME" x="-23.114" y="32.639" size="1.778" layer="95" rot="R180"/>
+<attribute name="VALUE" x="-18.161" y="32.004" size="1.778" layer="96" rot="R90"/>
+</instance>
+<instance part="C10" gate="G$1" x="2.54" y="96.52"/>
+<instance part="GND16" gate="1" x="2.54" y="86.36"/>
 </instances>
 <busses>
@@
 <pinref part="GND12" gate="1" pin="GND"/>
 <wire x1="-17.78" y1="121.92" x2="-17.78" y2="132.08" width="0.1524" layer="91"/>
-</segment>
-<segment>
-<pinref part="KRANC" gate="-2" pin="S"/>
-<wire x1="-10.16" y1="22.86" x2="2.54" y2="22.86" width="0.1524" layer="91"/>
-<label x="-7.62" y="22.86" size="1.778" layer="95"/>
-</segment>
-<segment>
-<pinref part="KRANC" gate="-3" pin="S"/>
-<wire x1="-10.16" y1="20.32" x2="2.54" y2="20.32" width="0.1524" layer="91"/>
-<label x="-7.62" y="20.32" size="1.778" layer="95"/>
 </segment>
 <segment>
@@
 <wire x1="205.74" y1="99.06" x2="210.82" y2="99.06" width="0.1524" layer="91"/>
 </segment>
+<segment>
+<pinref part="C1" gate="G$1" pin="1"/>
+<wire x1="-25.4" y1="30.48" x2="-35.56" y2="30.48" width="0.1524" layer="91"/>
+<label x="-35.56" y="30.48" size="1.778" layer="95"/>
+</segment>
+<segment>
+<pinref part="C10" gate="G$1" pin="2"/>
+<wire x1="2.54" y1="91.44" x2="2.54" y2="88.9" width="0.1524" layer="91"/>
+<pinref part="GND16" gate="1" pin="GND"/>
+</segment>
 </net>
 <net name="N$6" class="0">
@@
 </segment>
 <segment>
-<pinref part="R3" gate="G$1" pin="1"/>
-<wire x1="-25.4" y1="43.18" x2="-27.94" y2="43.18" width="0.1524" layer="91"/>
-<wire x1="-27.94" y1="43.18" x2="-27.94" y2="66.04" width="0.1524" layer="91"/>
-<pinref part="R2" gate="G$1" pin="1"/>
-<wire x1="-27.94" y1="66.04" x2="-5.08" y2="66.04" width="0.1524" layer="91"/>
-<pinref part="C4" gate="G$1" pin="1"/>
-<wire x1="-25.4" y1="38.1" x2="-27.94" y2="38.1" width="0.1524" layer="91"/>
-<wire x1="-27.94" y1="38.1" x2="-27.94" y2="43.18" width="0.1524" layer="91"/>
-<label x="-25.4" y="66.04" size="1.778" layer="95"/>
-</segment>
-<segment>
 <pinref part="ENKODER" gate="-1" pin="S"/>
 <wire x1="-10.16" y1="2.54" x2="2.54" y2="2.54" width="0.1524" layer="91"/>
@@
 <label x="-7.62" y="25.4" size="1.778" layer="95"/>
 </segment>
+<segment>
+<pinref part="UC" gate="G$1" pin="PC9/TIM3_CH4/TIM8_CH4(5T)"/>
+<wire x1="165.1" y1="66.04" x2="187.96" y2="66.04" width="0.1524" layer="91"/>
+<label x="175.26" y="66.04" size="1.778" layer="95"/>
+</segment>
 </net>
 <net name="MIN" class="0">
@@
 <wire x1="-10.16" y1="17.78" x2="2.54" y2="17.78" width="0.1524" layer="91"/>
 <label x="-7.62" y="17.78" size="1.778" layer="95"/>
+</segment>
+<segment>
+<pinref part="UC" gate="G$1" pin="PC8/TIM3_CH3/TIM8_CH3(5T)"/>
+<wire x1="165.1" y1="68.58" x2="187.96" y2="68.58" width="0.1524" layer="91"/>
+<label x="175.26" y="68.58" size="1.778" layer="95"/>
 </segment>
 </net>
@@
 <junction x="-5.08" y="48.26"/>
 <junction x="-5.08" y="43.18"/>
+<pinref part="C1" gate="G$1" pin="2"/>
+<wire x1="-17.78" y1="30.48" x2="-5.08" y2="30.48" width="0.1524" layer="91"/>
+<wire x1="-5.08" y1="30.48" x2="-5.08" y2="38.1" width="0.1524" layer="91"/>
+</segment>
+<segment>
+<pinref part="UC" gate="G$1" pin="PA10/TIM1_CH3/USART1_RX(5T)"/>
+<wire x1="78.74" y1="55.88" x2="71.12" y2="55.88" width="0.1524" layer="91"/>
+<label x="71.12" y="55.88" size="1.778" layer="95"/>
 </segment>
 </net>
@@
 <label x="-7.62" y="0" size="1.778" layer="95"/>
 </segment>
+<segment>
+<pinref part="UC" gate="G$1" pin="PA8/TIM1_CH1(5T)"/>
+<wire x1="78.74" y1="60.96" x2="71.12" y2="60.96" width="0.1524" layer="91"/>
+<label x="71.12" y="60.96" size="1.778" layer="95"/>
+</segment>
 </net>
 <net name="TOR2" class="0">
@@
 <label x="-7.62" y="-5.08" size="1.778" layer="95"/>
 </segment>
-</net>
-<net name="N$2" class="0">
-<segment>
-<pinref part="U$2" gate="G$1" pin="LED-"/>
-<wire x1="259.08" y1="10.16" x2="261.62" y2="10.16" width="0.1524" layer="91"/>
-<wire x1="261.62" y1="10.16" x2="261.62" y2="7.62" width="0.1524" layer="91"/>
-<pinref part="X3" gate="-1" pin="K"/>
-<wire x1="261.62" y1="7.62" x2="266.7" y2="7.62" width="0.1524" layer="91"/>
-</segment>
-</net>
-<net name="N$3" class="0">
-<segment>
-<pinref part="U$2" gate="G$1" pin="LED+"/>
-<wire x1="259.08" y1="12.7" x2="261.62" y2="12.7" width="0.1524" layer="91"/>
-<wire x1="261.62" y1="12.7" x2="261.62" y2="15.24" width="0.1524" layer="91"/>
-<pinref part="X3" gate="-2" pin="K"/>
-<wire x1="261.62" y1="15.24" x2="266.7" y2="15.24" width="0.1524" layer="91"/>
+<segment>
+<pinref part="UC" gate="G$1" pin="PA9/TIM1_CH2/USART1_TX(5T)"/>
+<wire x1="78.74" y1="58.42" x2="71.12" y2="58.42" width="0.1524" layer="91"/>
+<label x="71.12" y="58.42" size="1.778" layer="95"/>
 </segment>
 </net>
@@
 <pinref part="C2" gate="G$1" pin="1"/>
 <wire x1="-5.08" y1="101.6" x2="2.54" y2="101.6" width="0.1524" layer="91"/>
+<wire x1="2.54" y1="101.6" x2="5.08" y2="101.6" width="0.1524" layer="91"/>
 <wire x1="-5.08" y1="99.06" x2="-5.08" y2="101.6" width="0.1524" layer="91"/>
 <junction x="-5.08" y="101.6"/>
 <pinref part="IC2" gate="G$1" pin="OUT"/>
 <pinref part="+3V1" gate="G$1" pin="+3V3"/>
+<pinref part="C10" gate="G$1" pin="1"/>
+<wire x1="2.54" y1="99.06" x2="2.54" y2="101.6" width="0.1524" layer="91"/>
 </segment>
 <segment>
@@
 <wire x1="208.28" y1="127" x2="205.74" y2="127" width="0.1524" layer="91"/>
 <wire x1="205.74" y1="127" x2="205.74" y2="129.54" width="0.1524" layer="91"/>
+</segment>
+<segment>
+<pinref part="KRANC" gate="-2" pin="S"/>
+<wire x1="-10.16" y1="22.86" x2="2.54" y2="22.86" width="0.1524" layer="91"/>
+<label x="-7.62" y="22.86" size="1.778" layer="95"/>
+</segment>
+<segment>
+<pinref part="KRANC" gate="-3" pin="S"/>
+<wire x1="-10.16" y1="20.32" x2="2.54" y2="20.32" width="0.1524" layer="91"/>
+<label x="-7.62" y="20.32" size="1.778" layer="95"/>
+</segment>
+<segment>
+<pinref part="R2" gate="G$1" pin="1"/>
+<wire x1="-5.08" y1="66.04" x2="-5.08" y2="71.12" width="0.1524" layer="91"/>
+<wire x1="-5.08" y1="71.12" x2="-35.56" y2="71.12" width="0.1524" layer="91"/>
+<wire x1="-35.56" y1="71.12" x2="-35.56" y2="43.18" width="0.1524" layer="91"/>
+<pinref part="R3" gate="G$1" pin="1"/>
+<wire x1="-35.56" y1="43.18" x2="-25.4" y2="43.18" width="0.1524" layer="91"/>
+<wire x1="-35.56" y1="43.18" x2="-35.56" y2="38.1" width="0.1524" layer="91"/>
+<pinref part="C4" gate="G$1" pin="1"/>
+<wire x1="-35.56" y1="38.1" x2="-25.4" y2="38.1" width="0.1524" layer="91"/>
+<label x="-22.86" y="71.12" size="1.778" layer="95"/>
 </segment>
 </net>
@@
 </segment>
 </net>
+<net name="N$8" class="0">
+<segment>
+<pinref part="UC" gate="G$1" pin="PA11/TIM1_CH4/CANRX/USBDM(5T)"/>
+<wire x1="78.74" y1="53.34" x2="71.12" y2="53.34" width="0.1524" layer="91"/>
+</segment>
+</net>
+<net name="N$7" class="0">
+<segment>
+<pinref part="UC" gate="G$1" pin="PA12/CANTX/USBDP(5T)"/>
+<wire x1="78.74" y1="50.8" x2="71.12" y2="50.8" width="0.1524" layer="91"/>
+</segment>
+</net>

Commit message: 03-12-13 20:52
Parts:
- removed ENKODER, TRANS: MICROMATCH-4, con-maritex:MICROMATCH-4
- removed UC: STM32F405RGT, stm32f4:STM32F405R
- added ENC, T-OPT: MICROMATCH-4, con-maritex:MICROMATCH-4
- added U$1: STM32F405R, stm32f4:STM32F405R
- added UART: C-GRID-03-70543, con-molex:C-GRID-03-70543
Connections:
- removed net 1-ENA: U$4.ENA/DIAGA, UC.PC4/ADC12_IN14
- removed net 1-INA: U$4.INA, UC.PA7/TIM1_CH1N/ADC12_IN7(FT)
- removed net 1-PWM: U$4.PWM, UC.PC5/ADC12_IN15
- removed net N$10: U$4.ENB/DIAGB, UC.PB1/TIM1_CH3N/ADC12_IN9(5T)
- removed net N$11: U$4.CS, UC.PB0/TIM1_CH2N/ADC12_IN8(5T)
- removed net N$12: U$4.VOUT
- removed net N$13: U$3.INB, UC.PB12(5T)
- removed net N$15: U$3.PWM, UC.PB15/SPI2_MOSI(5T)
- removed net N$17: U$3.ENB/DIAGB, UC.PB13/SPI2_SCK(5T)
- removed net N$18: U$3.CS, UC.PB14/SPI2_MISO(5T)
- removed net N$19: U$3.VOUT
- removed net N$21: U$2.PWM
- removed net N$25: I2C-1.S
- removed net N$38: U$3.ENA/DIAGA, UC.PC6/TIM3_CH1/TIM_CH1/USART6_TX(5T)
- removed net N$39: U$3.INA, UC.PC7/TIM3_CH2/TIM8_CH2/USART6_RX(5T)
- removed net N$6: U$4.INB, UC.PB2/BOOT1(5T)
- removed net N$7: UC.PA12/CANTX/USBDP(5T)
- removed net N$8: UC.PA11/TIM1_CH4/CANRX/USBDM(5T)
- removed net TOR1: ENKODER-2.S, UC.PA8/TIM1_CH1(5T)
- removed net TOR2: ENKODER-4.S, UC.PA9/TIM1_CH2/USART1_TX(5T)
- new net ENC1: ENC-2.S, U$1.PA8
- new net ENC2: ENC-4.S, U$1.PA11
- new net LED-PWM: U$1.PB6, U$2.PWM
- new net M1-CS: U$1.PB0, U$4.CS
- new net M1-ENA: U$1.PC4, U$4.ENA/DIAGA
- new net M1-ENB: U$4.ENB/DIAGB
- new net M1-INA: U$1.PA7, U$4.INA
- new net M1-INB: U$4.INB
- new net M1-PWM: U$1.PC6, U$4.PWM
- new net M2-CS: U$1.PB1, U$3.CS
- new net M2-ENA: U$3.ENA/DIAGA
- new net M2-ENB: U$3.ENB/DIAGB
- new net M2-INA: U$3.INA
- new net M2-INB: U$3.INB
- new net M2-PWM: U$1.PC7, U$3.PWM
- new net RX: U$1.PA10, UART-2.S
- new net TX: U$1.PA9, UART-3.S
- net !JRST: now also U$1.PB4; no longer UC.PB4/JNTRST(5T)
- net !RST: now also U$1.NRST; no longer UC.NRST
- net +3V3: now also U$1.VDD_1, U$1.VDD_2, U$1.VDD_3, U$1.VDD_4; no longer UC.VDD_1, UC.VDD_2, UC.VDD_3, UC.VDD_4
- net +5V: now also ENC-1.S, I2C-4.S; no longer ENKODER-1.S
- net GND: now also ENC-3.S, I2C-3.S, T-OPT-2.S, T-OPT-3.S, U$1.BOOT0, U$1.VSSA, U$1.VSS_1, U$1.VSS_2, UART-1.S; no longer ENKODER-3.S, I2C-4.S, TRANS-2.S, TRANS-3.S, UC.BOOT0, UC.VSSA, UC.VSS_1, UC.VSS_2
- net JTCK: now also U$1.PA14; no longer UC.PA14/JTCK-SWCLK(5T)
- net JTDI: now also U$1.PA15; no longer UC.PA15/JTDI(5T)
- net JTDO: now also U$1.PB3; no longer UC.PB3/JTDO(5T)
- net JTMS: now also U$1.PA13; no longer UC.PA13/JTMS-SWDAT(5T)
- net MAX: no longer UC.PC9/TIM3_CH4/TIM8_CH4(5T)
- net MIN: no longer UC.PC8/TIM3_CH3/TIM8_CH3(5T)
- net N$1: now also T-OPT-1.S; no longer TRANS-1.S
- net N$20: now also U$1.VDDA; no longer UC.VDDA
- net N$22: now also U$1.OSC_OUT; no longer UC.PH1/OSC_OUT(5T)
- net N$23: now also U$1.VCAP_2; no longer UC.VCAP_2
- net N$24: now also U$1.VCAP_1; no longer UC.VCAP_1
- net N$5: now also U$1.OSC_IN; no longer UC.PH0/OSC_IN(5T)
- net SCL: now also I2C-2.S, U$1.PB10; no longer I2C-3.S, UC.PB10/I2C2_SCL(5T)
- net SDA: now also I2C-1.S, U$1.PB11; no longer I2C-2.S, UC.PB11/I2C2_SDA(5T)
- net TRANS: now also T-OPT-4.S; no longer TRANS-4.S, UC.PA10/TIM1_CH3/USART1_RX(5T)
Other:
- moved on the sheet: C1, C10, C2, C3, C4, C5, C6, C7, C8, C9, I2C-1, I2C-2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

Commit message: 11.12.13 18:50
Parts:
- added SV2: (no value), con-lstb:MA07-1
- IC2: value LD117AD2MTR -> LT1086CM-3.3
Connections:
- new net G_ADC1: SV2.3, U$1.PC0
- new net G_ADC2: SV2.4, U$1.PC1
- new net SRV1: SV2.5, U$1.PA8
- new net SRV2: SV2.6, U$1.PA11
- net +12V: now also SV2.7; no longer C3.1, IC2.IN
- net +5V: now also C3.1, IC2.IN, SV2.1
- net ENC1: now also U$1.PC6; no longer U$1.PA8
- net ENC2: now also U$1.PC7; no longer U$1.PA11
- net GND: now also SV2.2
- net LED-PWM: now also U$1.PC9; no longer U$1.PB6
- net M1-CS: now also U$1.PA2; no longer U$1.PB0
- net M1-ENA: now also U$1.PC3; no longer U$1.PC4
- net M1-ENB: now also U$1.PA3
- net M1-INA: now also U$1.PC2; no longer U$1.PA7
- net M1-INB: now also U$1.PA4
- net M1-PWM: now also U$1.PA1; no longer U$1.PC6
- net M2-CS: now also U$1.PA7; no longer U$1.PB1
- net M2-ENA: now also U$1.PB1
- net M2-ENB: now also U$1.PA6
- net M2-INA: now also U$1.PB2
- net M2-INB: now also U$1.PA5
- net M2-PWM: now also U$1.PB0; no longer U$1.PC7
- net MAX: now also U$1.PB11
- net MIN: now also U$1.PB10
- net SCL: now also U$1.PB8; no longer U$1.PB10
- net SDA: now also U$1.PB9; no longer U$1.PB11
- net TRANS: now also U$1.PC8
Other:
- note added: "(ADC123_IN2)"
- note added: "(ADC12_IN7)"
- note added: "(I2C1_SCL)"
- note added: "(I2C1_SDA)"
- note added: "(TIM2_CH2)"
- note added: "(TIM3_CH1)"
- note added: "(TIM3_CH2)"
- note added: "(TIM3_CH3)"
- note added: "(TIM3_CH4)"
- moved on the sheet: C7

Commit message: misc changes
Other:
- note added: "(USART1_RX)"
- note added: "(USART1_TX)"
Changed lines of the file:
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@@
 <wire x1="256.54" y1="175.26" x2="256.54" y2="208.28" width="0.1524" layer="97"/>
 <wire x1="256.54" y1="208.28" x2="226.06" y2="208.28" width="0.1524" layer="97"/>
-<text x="154.432" y="129.032" size="1.016" layer="96">(ADC12_IN7)</text>
+<text x="156.21" y="129.032" size="1.016" layer="96">(ADC12_IN7)</text>
 <text x="154.432" y="141.732" size="1.016" layer="96">(ADC123_IN2)</text>
 <text x="169.926" y="197.612" size="1.016" layer="96">(TIM3_CH3)</text>
@@
 <wire x1="223.52" y1="208.28" x2="223.52" y2="172.72" width="0.1524" layer="97"/>
 <wire x1="223.52" y1="172.72" x2="256.54" y2="172.72" width="0.1524" layer="97"/>
+<text x="156.21" y="123.952" size="1.016" layer="96">(USART1_TX)</text>
+<text x="156.21" y="121.412" size="1.016" layer="96">(USART1_RX)</text>
 </plain>
 <instances>
