File: mainb/mainb_v2/mainb_v2.sch (KiCad schematic (older format))
At the start: 23 parts, among them J1 RPI_GPIO, J2 ETH, Q1 BC337, Q2 BC337, U1 POLOLU-2111

Commit message: mainb: mainb_v2 kicad schematic updates
Parts:
- removed C?: C, ~, symbol C
- removed R?: R, ~, symbol R
- added BATT: CR2303, ~, symbol BATTERY
- added C? (x2): C, ~, symbol C
- added R1, R2, R?: ??, ~, symbol R
- added U2: ADS1110, ~, symbol ADS1110
- added U3: DS1307Z, ~, symbol DS1307Z
- gave numbers to parts that had none: 1
Connections:
- net labels added: AKU-, REL#1, REL#2, RX, SCL, SDA, TX
- wire segments 66 -> 122
Other:
- moved on the sheet: +12V relay, +5V relay, D1, D2, D3, D?, ETH->RPI, J1, J2, PoE relay, Q1, Q2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

Commit message: mainb: kicad sch updates
Parts:
- removed X: CRYSTAL, ~, symbol CRYSTAL
- added J10, J7, J8, J9: PWR, ~, symbol CONN_3
- added J3: I2C, ~, symbol CONN_4
- added J4, J5, J6: I2C, ~, symbol CONN_3
- added U4: MiniIMU-9, symbol MiniIMU-9
- added X1: CRYSTAL, ~, symbol CRYSTAL
- C1, C2: renamed from C?; value C -> 100n
- gave numbers to parts that had none: 5
- renumbered BATT to BATT1, ETH->RPI to ETH->RPI1, uart to J11, R3 to R7, R2 to R8, R1 to R9, +5V~relay to REL1, +12V~relay to REL2, PoE~relay to REL3
Connections:
- wire segments 122 -> 156
- no-connect marks 0 -> 8
Other:
- moved on the sheet: C1, C2, D1, D2, D3, D4, D5, J1, J11, Q1, Q2, R1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
