File: trinocular/rpicam/rpicam.sch (EAGLE design)
At the start: 9 parts, among them IC1 MEGA8-AI

Commit message: 03-12-13 20:52
Parts:
- removed U$2: RPICAM, RaspberryPi:RPICAM
- added LEDD#1, LEDD#2: (no value), con-lstb:MA04-1
- added SRV: power, con-molex:C-GRID-03-70543
Connections:
- removed net N$3: I2C-3.S
- removed net N$5: I2C-4.S
- removed net N$9: R1.2, U$1.A
- new net SCL: I2C-2.S, IC1.PC5(ADC5/SCL)
- new net SDA: I2C-1.S, IC1.PC4(ADC4/SDA)
- net +12V: now also LEDD#1.3, LEDD#2.3
- net +5V: now also I2C-4.S, LEDD#1.1, LEDD#2.1, U$1.A; no longer U$1.C
- net GND: now also I2C-3.S, LEDD#1.4, LEDD#2.4, SRV-3.S
- net LED1_CTRL: now also LEDD#1.2
- net LED2_CTRL: now also LEDD#2.2
- net MOSI/SRV_CTRL: now also SRV-1.S
- net N$1: now also R1.2, U$1.C; no longer I2C-1.S
- net N$2: now also SRV-2.S; no longer I2C-2.S
Changed lines of the file:
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@@
 <?xml version="1.0" encoding="utf-8"?>
 <!DOCTYPE eagle SYSTEM "eagle.dtd">
-<eagle version="6.1">
+<eagle version="6.4">
 <drawing>
 <settings>
@@
 <part name="R1" library="rcl" deviceset="R-EU_" device="R0603"/>
 <part name="C1" library="rcl" deviceset="C-EU" device="C0603"/>
-<part name="U$2" library="RaspberryPi" deviceset="RPICAM" device=""/>
+<part name="P+3" library="supply1" deviceset="+5V" device=""/>
+<part name="GND3" library="supply1" deviceset="GND" device=""/>
+<part name="LEDD#1" library="con-lstb" deviceset="MA04-1" device=""/>
+<part name="LEDD#2" library="con-lstb" deviceset="MA04-1" device=""/>
+<part name="P+6" library="supply1" deviceset="+5V" device=""/>
+<part name="GND4" library="supply1" deviceset="GND" device=""/>
+<part name="P+7" library="supply1" deviceset="+12V" device=""/>
+<part name="P+8" library="supply1" deviceset="+5V" device=""/>
+<part name="GND6" library="supply1" deviceset="GND" device=""/>
+<part name="SRV" library="con-molex" deviceset="C-GRID-03" device="-70543" value="power"/>
 </parts>
 <sheets>
@@
 <instance part="GND1" gate="1" x="38.1" y="167.64" rot="MR0"/>
 <instance part="GND2" gate="1" x="43.18" y="149.86" rot="MR0"/>
-<instance part="I2C" gate="-1" x="30.48" y="101.6"/>
+<instance part="I2C" gate="-1" x="30.48" y="101.6" smashed="yes">
+<attribute name="NAME" x="29.972" y="102.489" size="1.778" layer="95" rot="R180"/>
+</instance>
 <instance part="I2C" gate="-2" x="30.48" y="99.06"/>
 <instance part="I2C" gate="-3" x="30.48" y="96.52"/>
@@
 </instance>
 <instance part="PWR" gate="-3" x="27.94" y="172.72" rot="MR0"/>
-<instance part="U$1" gate="G$1" x="170.18" y="177.8" smashed="yes"/>
+<instance part="U$1" gate="G$1" x="170.18" y="177.8" smashed="yes" rot="MR0"/>
 <instance part="R1" gate="G$1" x="160.02" y="177.8"/>
 <instance part="C1" gate="G$1" x="93.98" y="144.78"/>
-<instance part="U$2" gate="G$1" x="33.02" y="76.2"/>
+<instance part="P+3" gate="1" x="55.88" y="93.98" rot="R270"/>
+<instance part="GND3" gate="1" x="45.72" y="86.36"/>
+<instance part="LEDD#1" gate="1" x="213.36" y="96.52" rot="R180"/>
+<instance part="LEDD#2" gate="1" x="213.36" y="76.2" rot="R180"/>
+<instance part="P+6" gate="1" x="198.12" y="109.22" rot="MR0"/>
+<instance part="GND4" gate="1" x="200.66" y="63.5"/>
+<instance part="P+7" gate="1" x="193.04" y="109.22"/>
+<instance part="P+8" gate="1" x="203.2" y="134.62" smashed="yes">
+<attribute name="VALUE" x="205.74" y="137.16" size="1.778" layer="96" rot="R180"/>
+</instance>
+<instance part="GND6" gate="1" x="203.2" y="116.84"/>
+<instance part="SRV" gate="-1" x="208.28" y="124.46" smashed="yes" rot="MR180">
+<attribute name="NAME" x="210.82" y="125.222" size="1.524" layer="95" rot="MR180"/>
+</instance>
+<instance part="SRV" gate="-2" x="208.28" y="127" rot="MR180"/>
+<instance part="SRV" gate="-3" x="208.28" y="121.92" rot="MR180"/>
 </instances>
 <busses>
@@
 <nets>
 <net name="+5V" class="0">
-<segment>
-<pinref part="P+4" gate="1" pin="+5V"/>
-<pinref part="U$1" gate="G$1" pin="C"/>
-<wire x1="172.72" y1="177.8" x2="177.8" y2="177.8" width="0.1524" layer="91"/>
-</segment>
 <segment>
 <wire x1="104.14" y1="167.64" x2="91.44" y2="167.64" width="0.1524" layer="91"/>
@@
 <pinref part="PWR" gate="-1" pin="S"/>
 </segment>
+<segment>
+<pinref part="I2C" gate="-4" pin="S"/>
+<wire x1="35.56" y1="93.98" x2="53.34" y2="93.98" width="0.1524" layer="91"/>
+<pinref part="P+3" gate="1" pin="+5V"/>
+</segment>
+<segment>
+<pinref part="LEDD#1" gate="1" pin="1"/>
+<pinref part="P+6" gate="1" pin="+5V"/>
+<wire x1="205.74" y1="101.6" x2="198.12" y2="101.6" width="0.1524" layer="91"/>
+<wire x1="198.12" y1="101.6" x2="198.12" y2="106.68" width="0.1524" layer="91"/>
+<pinref part="LEDD#2" gate="1" pin="1"/>
+<wire x1="205.74" y1="81.28" x2="198.12" y2="81.28" width="0.1524" layer="91"/>
+<wire x1="198.12" y1="81.28" x2="198.12" y2="101.6" width="0.1524" layer="91"/>
+<junction x="198.12" y="101.6"/>
+</segment>
+<segment>
+<pinref part="P+8" gate="1" pin="+5V"/>
+<wire x1="203.2" y1="129.54" x2="203.2" y2="132.08" width="0.1524" layer="91"/>
+</segment>
+<segment>
+<pinref part="U$1" gate="G$1" pin="A"/>
+<pinref part="P+4" gate="1" pin="+5V"/>
+<wire x1="172.72" y1="177.8" x2="177.8" y2="177.8" width="0.1524" layer="91"/>
+</segment>
 </net>
 <net name="GND" class="0">
@@
 <pinref part="PWR" gate="-2" pin="S"/>
 </segment>
+<segment>
+<pinref part="I2C" gate="-3" pin="S"/>
+<wire x1="35.56" y1="96.52" x2="45.72" y2="96.52" width="0.1524" layer="91"/>
+<pinref part="GND3" gate="1" pin="GND"/>
+<wire x1="45.72" y1="88.9" x2="45.72" y2="96.52" width="0.1524" layer="91"/>
+</segment>
+<segment>
+<pinref part="LEDD#1" gate="1" pin="4"/>
+<pinref part="GND4" gate="1" pin="GND"/>
+<wire x1="205.74" y1="93.98" x2="200.66" y2="93.98" width="0.1524" layer="91"/>
+<wire x1="200.66" y1="93.98" x2="200.66" y2="73.66" width="0.1524" layer="91"/>
+<pinref part="LEDD#2" gate="1" pin="4"/>
+<wire x1="200.66" y1="73.66" x2="200.66" y2="66.04" width="0.1524" layer="91"/>
+<wire x1="205.74" y1="73.66" x2="200.66" y2="73.66" width="0.1524" layer="91"/>
+</segment>
+<segment>
+<pinref part="GND6" gate="1" pin="GND"/>
+<wire x1="203.2" y1="121.92" x2="203.2" y2="119.38" width="0.1524" layer="91"/>
+<pinref part="SRV" gate="-3" pin="S"/>
+<wire x1="203.2" y1="121.92" x2="205.74" y2="121.92" width="0.1524" layer="91"/>
+</segment>
 </net>
 <net name="RST" class="0">
@@
 </segment>
 </net>
-<net name="N$9" class="0">
-<segment>
-<wire x1="167.64" y1="177.8" x2="165.1" y2="177.8" width="0.1524" layer="91"/>
-<pinref part="U$1" gate="G$1" pin="A"/>
-<pinref part="R1" gate="G$1" pin="2"/>
-</segment>
-</net>
 <net name="RXD" class="0">
 <segment>
@@
 <pinref part="PWR" gate="-3" pin="S"/>
 </segment>
+<segment>
+<pinref part="LEDD#1" gate="1" pin="3"/>
+<pinref part="P+7" gate="1" pin="+12V"/>
+<wire x1="205.74" y1="96.52" x2="193.04" y2="96.52" width="0.1524" layer="91"/>
+<wire x1="193.04" y1="96.52" x2="193.04" y2="106.68" width="0.1524" layer="91"/>
+<pinref part="LEDD#2" gate="1" pin="3"/>
+<wire x1="205.74" y1="76.2" x2="193.04" y2="76.2" width="0.1524" layer="91"/>
+<wire x1="193.04" y1="76.2" x2="193.04" y2="96.52" width="0.1524" layer="91"/>
+<junction x="193.04" y="96.52"/>
+</segment>
 </net>
 <net name="LED2_CTRL" class="0">
@@
 <pinref part="IC1" gate="G$1" pin="PB2(SS/OC1B)"/>
 </segment>
+<segment>
+<pinref part="LEDD#2" gate="1" pin="2"/>
+<wire x1="205.74" y1="78.74" x2="175.26" y2="78.74" width="0.1524" layer="91"/>
+<label x="175.26" y="78.994" size="1.778" layer="95"/>
+</segment>
 </net>
 <net name="LED1_CTRL" class="0">
@@
 <pinref part="IC1" gate="G$1" pin="PB1(OC1A)"/>
 </segment>
-</net>
-<net name="N$1" class="0">
+<segment>
+<pinref part="LEDD#1" gate="1" pin="2"/>
+<wire x1="205.74" y1="99.06" x2="175.26" y2="99.06" width="0.1524" layer="91"/>
+<label x="175.26" y="99.314" size="1.778" layer="95"/>
+</segment>
+</net>
+<net name="SDA" class="0">
 <segment>
 <pinref part="I2C" gate="-1" pin="S"/>
 <wire x1="35.56" y1="101.6" x2="45.72" y2="101.6" width="0.1524" layer="91"/>
-</segment>
-</net>
-<net name="N$2" class="0">
+<label x="40.64" y="101.854" size="1.778" layer="95"/>
+</segment>
+<segment>
+<pinref part="IC1" gate="G$1" pin="PC4(ADC4/SDA)"/>
+<wire x1="152.4" y1="167.64" x2="162.56" y2="167.64" width="0.1524" layer="91"/>
+<label x="157.988" y="167.894" size="1.778" layer="95"/>
+</segment>
+</net>
+<net name="SCL" class="0">
 <segment>
 <pinref part="I2C" gate="-2" pin="S"/>
 <wire x1="35.56" y1="99.06" x2="45.72" y2="99.06" width="0.1524" layer="91"/>
-</segment>
-</net>
-<net name="N$3" class="0">
-<segment>
-<pinref part="I2C" gate="-3" pin="S"/>
-<wire x1="35.56" y1="96.52" x2="45.72" y2="96.52" width="0.1524" layer="91"/>
-</segment>
-</net>
-<net name="N$5" class="0">
-<segment>
-<pinref part="I2C" gate="-4" pin="S"/>
-<wire x1="35.56" y1="93.98" x2="45.72" y2="93.98" width="0.1524" layer="91"/>
+<label x="40.64" y="99.314" size="1.778" layer="95"/>
+</segment>
+<segment>
+<pinref part="IC1" gate="G$1" pin="PC5(ADC5/SCL)"/>
+<wire x1="152.4" y1="165.1" x2="162.56" y2="165.1" width="0.1524" layer="91"/>
+<label x="157.988" y="165.354" size="1.778" layer="95"/>
 </segment>
 </net>
 <net name="MOSI/SRV_CTRL" class="0">
 <segment>
-<wire x1="152.4" y1="124.46" x2="170.18" y2="124.46" width="0.1524" layer="91"/>
-<label x="156.718" y="124.714" size="1.778" layer="95"/>
+<label x="171.958" y="124.714" size="1.778" layer="95"/>
 <pinref part="IC1" gate="G$1" pin="PB3(MOSI/OC2)"/>
+<wire x1="152.4" y1="124.46" x2="205.74" y2="124.46" width="0.1524" layer="91"/>
+<pinref part="SRV" gate="-1" pin="S"/>
 </segment>
 <segment>
@@
 </segment>
 </net>
+<net name="N$1" class="0">
+<segment>
+<pinref part="R1" gate="G$1" pin="2"/>
+<pinref part="U$1" gate="G$1" pin="C"/>
+<wire x1="165.1" y1="177.8" x2="167.64" y2="177.8" width="0.1524" layer="91"/>
+</segment>
+</net>
+<net name="N$2" class="0">
+<segment>
+<pinref part="SRV" gate="-2" pin="S"/>
+<wire x1="203.2" y1="129.54" x2="203.2" y2="127" width="0.1524" layer="91"/>
+<wire x1="203.2" y1="127" x2="205.74" y2="127" width="0.1524" layer="91"/>
+</segment>
+</net>

Commit message: 11.12.13 18:50
Parts:
- removed LEDD#1, LEDD#2: (no value), con-lstb:MA04-1
- removed PWR: power, con-molex:C-GRID-03-70543
Connections:
- removed net +12V: LEDD#1.3, LEDD#2.3, PWR-3.S
- removed net N$2: SRV-2.S
- net +5V: now also SRV-2.S; no longer LEDD#1.1, LEDD#2.1, PWR-1.S
- net GND: no longer LEDD#1.4, LEDD#2.4, PWR-2.S
- net LED1_CTRL: no longer LEDD#1.2
- net LED2_CTRL: no longer LEDD#2.2
Changed lines of the file:
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@@
 <?xml version="1.0" encoding="utf-8"?>
 <!DOCTYPE eagle SYSTEM "eagle.dtd">
-<eagle version="6.4">
+<eagle version="6.1">
 <drawing>
 <settings>
@@
 <part name="P+5" library="supply1" deviceset="+5V" device=""/>
 <part name="GND5" library="supply1" deviceset="GND" device=""/>
-<part name="P+1" library="supply1" deviceset="+12V" device=""/>
-<part name="P+2" library="supply1" deviceset="+5V" device=""/>
-<part name="GND1" library="supply1" deviceset="GND" device=""/>
 <part name="GND2" library="supply1" deviceset="GND" device=""/>
 <part name="I2C" library="con-amp-micromatch" deviceset="MICROMATCH-4" device=""/>
 <part name="UART" library="con-molex" deviceset="C-GRID-03" device="-70543" value="uart"/>
-<part name="PWR" library="con-molex" deviceset="C-GRID-03" device="-70543" value="power"/>
 <part name="U$1" library="wb" deviceset="LED0603" device=""/>
 <part name="R1" library="rcl" deviceset="R-EU_" device="R0603"/>
@@
 <part name="P+3" library="supply1" deviceset="+5V" device=""/>
 <part name="GND3" library="supply1" deviceset="GND" device=""/>
-<part name="LEDD#1" library="con-lstb" deviceset="MA04-1" device=""/>
-<part name="LEDD#2" library="con-lstb" deviceset="MA04-1" device=""/>
-<part name="P+6" library="supply1" deviceset="+5V" device=""/>
-<part name="GND4" library="supply1" deviceset="GND" device=""/>
-<part name="P+7" library="supply1" deviceset="+12V" device=""/>
 <part name="P+8" library="supply1" deviceset="+5V" device=""/>
 <part name="GND6" library="supply1" deviceset="GND" device=""/>
@@
 <instance part="P+5" gate="1" x="48.26" y="129.54" rot="R270"/>
 <instance part="GND5" gate="1" x="45.72" y="116.84"/>
-<instance part="P+1" gate="1" x="45.72" y="172.72" rot="MR90"/>
-<instance part="P+2" gate="1" x="45.72" y="177.8" rot="R270"/>
-<instance part="GND1" gate="1" x="38.1" y="167.64" rot="MR0"/>
 <instance part="GND2" gate="1" x="43.18" y="149.86" rot="MR0"/>
 <instance part="I2C" gate="-1" x="30.48" y="101.6" smashed="yes">
@@
 <attribute name="NAME" x="25.4" y="149.098" size="1.524" layer="95" rot="MR0"/>
 </instance>
-<instance part="PWR" gate="-1" x="27.94" y="177.8" smashed="yes" rot="MR0">
-<attribute name="NAME" x="25.4" y="177.038" size="1.524" layer="95" rot="MR0"/>
-</instance>
-<instance part="PWR" gate="-2" x="27.94" y="175.26" smashed="yes" rot="MR0">
-<attribute name="NAME" x="25.4" y="174.498" size="1.524" layer="95" rot="MR0"/>
-</instance>
-<instance part="PWR" gate="-3" x="27.94" y="172.72" rot="MR0"/>
 <instance part="U$1" gate="G$1" x="170.18" y="177.8" smashed="yes" rot="MR0"/>
 <instance part="R1" gate="G$1" x="160.02" y="177.8"/>
@@
 <instance part="P+3" gate="1" x="55.88" y="93.98" rot="R270"/>
 <instance part="GND3" gate="1" x="45.72" y="86.36"/>
-<instance part="LEDD#1" gate="1" x="213.36" y="96.52" rot="R180"/>
-<instance part="LEDD#2" gate="1" x="213.36" y="76.2" rot="R180"/>
-<instance part="P+6" gate="1" x="198.12" y="109.22" rot="MR0"/>
-<instance part="GND4" gate="1" x="200.66" y="63.5"/>
-<instance part="P+7" gate="1" x="193.04" y="109.22"/>
 <instance part="P+8" gate="1" x="203.2" y="134.62" smashed="yes">
 <attribute name="VALUE" x="205.74" y="137.16" size="1.778" layer="96" rot="R180"/>
@@
 </segment>
 <segment>
-<pinref part="P+2" gate="1" pin="+5V"/>
-<wire x1="30.48" y1="177.8" x2="43.18" y2="177.8" width="0.1524" layer="91"/>
-<pinref part="PWR" gate="-1" pin="S"/>
-</segment>
-<segment>
 <pinref part="I2C" gate="-4" pin="S"/>
 <wire x1="35.56" y1="93.98" x2="53.34" y2="93.98" width="0.1524" layer="91"/>
@@
 </segment>
 <segment>
-<pinref part="LEDD#1" gate="1" pin="1"/>
-<pinref part="P+6" gate="1" pin="+5V"/>
-<wire x1="205.74" y1="101.6" x2="198.12" y2="101.6" width="0.1524" layer="91"/>
-<wire x1="198.12" y1="101.6" x2="198.12" y2="106.68" width="0.1524" layer="91"/>
-<pinref part="LEDD#2" gate="1" pin="1"/>
-<wire x1="205.74" y1="81.28" x2="198.12" y2="81.28" width="0.1524" layer="91"/>
-<wire x1="198.12" y1="81.28" x2="198.12" y2="101.6" width="0.1524" layer="91"/>
-<junction x="198.12" y="101.6"/>
-</segment>
-<segment>
-<pinref part="P+8" gate="1" pin="+5V"/>
-<wire x1="203.2" y1="129.54" x2="203.2" y2="132.08" width="0.1524" layer="91"/>
-</segment>
-<segment>
 <pinref part="U$1" gate="G$1" pin="A"/>
 <pinref part="P+4" gate="1" pin="+5V"/>
 <wire x1="172.72" y1="177.8" x2="177.8" y2="177.8" width="0.1524" layer="91"/>
+</segment>
+<segment>
+<pinref part="SRV" gate="-2" pin="S"/>
+<wire x1="203.2" y1="127" x2="205.74" y2="127" width="0.1524" layer="91"/>
+<pinref part="P+8" gate="1" pin="+5V"/>
+<wire x1="203.2" y1="132.08" x2="203.2" y2="127" width="0.1524" layer="91"/>
 </segment>
 </net>
@@
 </segment>
 <segment>
-<pinref part="GND1" gate="1" pin="GND"/>
-<wire x1="30.48" y1="175.26" x2="38.1" y2="175.26" width="0.1524" layer="91"/>
-<wire x1="38.1" y1="175.26" x2="38.1" y2="170.18" width="0.1524" layer="91"/>
-<pinref part="PWR" gate="-2" pin="S"/>
-</segment>
-<segment>
 <pinref part="I2C" gate="-3" pin="S"/>
 <wire x1="35.56" y1="96.52" x2="45.72" y2="96.52" width="0.1524" layer="91"/>
@@
 </segment>
 <segment>
-<pinref part="LEDD#1" gate="1" pin="4"/>
-<pinref part="GND4" gate="1" pin="GND"/>
-<wire x1="205.74" y1="93.98" x2="200.66" y2="93.98" width="0.1524" layer="91"/>
-<wire x1="200.66" y1="93.98" x2="200.66" y2="73.66" width="0.1524" layer="91"/>
-<pinref part="LEDD#2" gate="1" pin="4"/>
-<wire x1="200.66" y1="73.66" x2="200.66" y2="66.04" width="0.1524" layer="91"/>
-<wire x1="205.74" y1="73.66" x2="200.66" y2="73.66" width="0.1524" layer="91"/>
-</segment>
-<segment>
 <pinref part="GND6" gate="1" pin="GND"/>
 <wire x1="203.2" y1="121.92" x2="203.2" y2="119.38" width="0.1524" layer="91"/>
@@
 </segment>
 </net>
-<net name="+12V" class="0">
-<segment>
-<pinref part="P+1" gate="1" pin="+12V"/>
-<wire x1="30.48" y1="172.72" x2="43.18" y2="172.72" width="0.1524" layer="91"/>
-<pinref part="PWR" gate="-3" pin="S"/>
-</segment>
-<segment>
-<pinref part="LEDD#1" gate="1" pin="3"/>
-<pinref part="P+7" gate="1" pin="+12V"/>
-<wire x1="205.74" y1="96.52" x2="193.04" y2="96.52" width="0.1524" layer="91"/>
-<wire x1="193.04" y1="96.52" x2="193.04" y2="106.68" width="0.1524" layer="91"/>
-<pinref part="LEDD#2" gate="1" pin="3"/>
-<wire x1="205.74" y1="76.2" x2="193.04" y2="76.2" width="0.1524" layer="91"/>
-<wire x1="193.04" y1="76.2" x2="193.04" y2="96.52" width="0.1524" layer="91"/>
-<junction x="193.04" y="96.52"/>
-</segment>
-</net>
 <net name="LED2_CTRL" class="0">
 <segment>
@@
 <pinref part="IC1" gate="G$1" pin="PB2(SS/OC1B)"/>
 </segment>
-<segment>
-<pinref part="LEDD#2" gate="1" pin="2"/>
-<wire x1="205.74" y1="78.74" x2="175.26" y2="78.74" width="0.1524" layer="91"/>
-<label x="175.26" y="78.994" size="1.778" layer="95"/>
-</segment>
 </net>
 <net name="LED1_CTRL" class="0">
@@
 <label x="157.734" y="129.794" size="1.778" layer="95"/>
 <pinref part="IC1" gate="G$1" pin="PB1(OC1A)"/>
-</segment>
-<segment>
-<pinref part="LEDD#1" gate="1" pin="2"/>
-<wire x1="205.74" y1="99.06" x2="175.26" y2="99.06" width="0.1524" layer="91"/>
-<label x="175.26" y="99.314" size="1.778" layer="95"/>
 </segment>
 </net>
@@
 </segment>
 </net>
-<net name="N$2" class="0">
-<segment>
-<pinref part="SRV" gate="-2" pin="S"/>
-<wire x1="203.2" y1="129.54" x2="203.2" y2="127" width="0.1524" layer="91"/>
-<wire x1="203.2" y1="127" x2="205.74" y2="127" width="0.1524" layer="91"/>
-</segment>
-</net>

Commit message: trinocular: rpicam hw revisions in single files
Parts:
- removed I2C: MICROMATCH-4, con-amp-micromatch:MICROMATCH-4
- removed SRV: power, con-molex:C-GRID-03-70543
- added SV1: (no value), con-lstb:MA20-2
- added SV2, SV3: (no value), con-lstb:MA04-1
- added X1: C-GRID-03-70553, con-molex:C-GRID-03-70553
- added X2: (no value), con-ptr500:AK500/2
- UART: device con-molex:C-GRID-03-70543 -> con-molex:C-GRID-03-70553
Connections:
- net +5V: now also SV1.2, SV1.4, SV2.1, SV2.3, SV3.1, SV3.3, X1-2.S, X2-1.KL; no longer I2C-4.S, SRV-2.S
- net GND: now also SV1.14, SV1.20, SV1.25, SV1.30, SV1.34, SV1.39, SV1.6, SV1.9, SV2.4, SV3.4, X1-3.S, X2-2.KL; no longer I2C-3.S, SRV-3.S
- net LED1_CTRL: now also SV2.2
- net LED2_CTRL: now also SV3.2
- net MOSI/SRV_CTRL: now also X1-1.S; no longer SRV-1.S
- net SCL: now also SV1.5; no longer I2C-2.S
- net SDA: now also SV1.3; no longer I2C-1.S
