File: trinocular/pcb/rpicam.sch (EAGLE design)
At the start: 11 parts, among them IC1 MEGA8-AI, X1 C-GRID-03-70553

Commit message: trinocular: PCB rev.3 - wip
Parts:
- removed SV3: (no value), con-lstb:MA04-1
- removed U$1: LED0603, wb:LED0603
- added I2C: MICROMATCH-4, con-maritex:MICROMATCH-4
- added LED1: (no value), led:LEDCHIP-LED0805
- C1: device rcl:C-EUC0603 -> rcl:C-EUC0805
- R1: device rcl:R-EU_R0603 -> rcl:R-EU_R0805
- SV1: device con-lstb:MA20-2 -> con-lstb:MA04-1
Connections:
- new net +18V: SV1.2, SV2.2, X2-1.KL
- net +5V: now also I2C-4.S, LED1.A, SV2.4; no longer SV1.2, SV2.1, SV2.3, SV3.1, SV3.3, U$1.A, X2-1.KL
- net GND: now also I2C-3.S, SV1.1, SV2.1; no longer SV1.14, SV1.20, SV1.25, SV1.30, SV1.34, SV1.39, SV1.6, SV1.9, SV2.4, SV3.4
- net LED1_CTRL: now also SV1.3; no longer SV2.2
- net LED2_CTRL: now also SV2.3; no longer SV3.2
- net N$1: now also LED1.C; no longer U$1.C
- net SCL: now also I2C-2.S; no longer SV1.5
- net SDA: now also I2C-1.S; no longer SV1.3
Other:
- note added: "TODO: - light sensor conn. - LED ctrl. connectors (2) - camera hole"
- moved on the sheet: SV2

Commit message: trinocular: PCB v3 - wip
Parts:
- removed I2C: MICROMATCH-4, con-maritex:MICROMATCH-4
- removed UART: uart, con-molex:C-GRID-03-70553
- added SV3: (no value), con-lstb:MA03-2
- added SV4: (no value), con-lstb:MA03-1
Connections:
- net +5V: now also SV3.4; no longer I2C-4.S
- net GND: now also SV3.3, SV4.1; no longer I2C-3.S, UART-1.S
- net RXD: now also SV4.2; no longer UART-2.S
- net SCL: now also SV3.2; no longer I2C-2.S
- net SDA: now also SV3.1; no longer I2C-1.S
- net TXD: now also SV4.3; no longer UART-3.S
Changed lines of the file:
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@@
 <part name="GND5" library="supply1" deviceset="GND" device=""/>
 <part name="GND2" library="supply1" deviceset="GND" device=""/>
-<part name="UART" library="con-molex" deviceset="C-GRID-03" device="-70553" value="uart"/>
 <part name="R1" library="rcl" deviceset="R-EU_" device="R0805"/>
 <part name="C1" library="rcl" deviceset="C-EU" device="C0805"/>
@@
 <part name="GND8" library="supply1" deviceset="GND" device=""/>
 <part name="P+3" library="supply1" deviceset="+18V" device=""/>
-<part name="I2C" library="con-maritex" deviceset="MICROMATCH-4" device="" value=""/>
 <part name="GND15" library="supply1" deviceset="GND" device=""/>
 <part name="P+7" library="supply1" deviceset="+5V" device=""/>
@@
 <part name="GND3" library="supply1" deviceset="GND" device=""/>
 <part name="LED1" library="led" deviceset="LED" device="CHIP-LED0805"/>
+<part name="SV3" library="con-lstb" deviceset="MA03-2" device=""/>
+<part name="SV4" library="con-lstb" deviceset="MA03-1" device=""/>
 </parts>
 <sheets>
@@
 <instance part="GND5" gate="1" x="45.72" y="116.84"/>
 <instance part="GND2" gate="1" x="43.18" y="149.86" rot="MR0"/>
-<instance part="UART" gate="-1" x="27.94" y="154.94" smashed="yes" rot="MR0">
-<attribute name="NAME" x="25.4" y="154.178" size="1.524" layer="95" rot="MR0"/>
-</instance>
-<instance part="UART" gate="-2" x="27.94" y="152.4" smashed="yes" rot="MR0">
-<attribute name="NAME" x="25.4" y="151.638" size="1.524" layer="95" rot="MR0"/>
-</instance>
-<instance part="UART" gate="-3" x="27.94" y="149.86" smashed="yes" rot="MR0">
-<attribute name="NAME" x="25.4" y="149.098" size="1.524" layer="95" rot="MR0"/>
-</instance>
 <instance part="R1" gate="G$1" x="160.02" y="177.8"/>
 <instance part="C1" gate="G$1" x="93.98" y="144.78"/>
@@
 <instance part="GND8" gate="1" x="33.02" y="167.64" rot="MR0"/>
 <instance part="P+3" gate="1" x="33.02" y="185.42"/>
-<instance part="I2C" gate="-1" x="52.07" y="78.74" smashed="yes">
-<attribute name="NAME" x="51.562" y="79.502" size="1.524" layer="95" rot="R180"/>
-</instance>
-<instance part="I2C" gate="-2" x="52.07" y="81.28"/>
-<instance part="I2C" gate="-3" x="52.07" y="83.82"/>
-<instance part="I2C" gate="-4" x="52.07" y="76.2"/>
-<instance part="GND15" gate="1" x="59.69" y="88.9" rot="R180"/>
-<instance part="P+7" gate="1" x="59.69" y="71.12" smashed="yes" rot="R180">
-<attribute name="VALUE" x="57.15" y="68.58" size="1.778" layer="96"/>
+<instance part="GND15" gate="1" x="64.77" y="55.88" rot="MR0"/>
+<instance part="P+7" gate="1" x="35.56" y="68.58" smashed="yes" rot="MR0">
+<attribute name="VALUE" x="33.02" y="71.12" size="1.778" layer="96" rot="MR180"/>
 </instance>
 <instance part="SV1" gate="1" x="109.22" y="81.28"/>
@@
 <attribute name="VALUE" x="168.148" y="172.085" size="1.778" layer="96"/>
 </instance>
+<instance part="SV3" gate="1" x="48.26" y="60.96"/>
+<instance part="SV4" gate="G$1" x="22.86" y="152.4" rot="MR180"/>
 </instances>
 <busses>
@@
 </segment>
 <segment>
-<pinref part="I2C" gate="-4" pin="S"/>
-<pinref part="P+7" gate="1" pin="+5V"/>
-<wire x1="57.15" y1="76.2" x2="59.69" y2="76.2" width="0.1524" layer="91"/>
-<wire x1="59.69" y1="76.2" x2="59.69" y2="73.66" width="0.1524" layer="91"/>
-</segment>
-<segment>
 <pinref part="SV1" gate="1" pin="4"/>
 <pinref part="P+9" gate="1" pin="+5V"/>
@@
 <wire x1="116.84" y1="50.8" x2="119.38" y2="50.8" width="0.1524" layer="91"/>
 <wire x1="119.38" y1="50.8" x2="119.38" y2="55.88" width="0.1524" layer="91"/>
+</segment>
+<segment>
+<pinref part="SV3" gate="1" pin="4"/>
+<wire x1="40.64" y1="60.96" x2="35.56" y2="60.96" width="0.1524" layer="91"/>
+<pinref part="P+7" gate="1" pin="+5V"/>
+<wire x1="35.56" y1="66.04" x2="35.56" y2="60.96" width="0.1524" layer="91"/>
 </segment>
 </net>
@@
 </segment>
 <segment>
-<wire x1="30.48" y1="154.94" x2="43.18" y2="154.94" width="0.1524" layer="91"/>
 <label x="33.02" y="154.94" size="1.778" layer="95"/>
 <pinref part="GND2" gate="1" pin="GND"/>
+<wire x1="30.48" y1="154.94" x2="43.18" y2="154.94" width="0.1524" layer="91"/>
 <wire x1="43.18" y1="154.94" x2="43.18" y2="152.4" width="0.1524" layer="91"/>
-<pinref part="UART" gate="-1" pin="S"/>
+<pinref part="SV4" gate="G$1" pin="1"/>
 </segment>
 <segment>
@@
 <segment>
 <pinref part="GND15" gate="1" pin="GND"/>
-<wire x1="59.69" y1="86.36" x2="59.69" y2="83.82" width="0.1524" layer="91"/>
-<wire x1="59.69" y1="83.82" x2="57.15" y2="83.82" width="0.1524" layer="91"/>
-<pinref part="I2C" gate="-3" pin="S"/>
+<wire x1="64.77" y1="58.42" x2="64.77" y2="60.96" width="0.1524" layer="91"/>
+<pinref part="SV3" gate="1" pin="3"/>
+<wire x1="55.88" y1="60.96" x2="64.77" y2="60.96" width="0.1524" layer="91"/>
 </segment>
 <segment>
@@
 </segment>
 <segment>
-<wire x1="30.48" y1="152.4" x2="38.1" y2="152.4" width="0.1524" layer="91"/>
 <label x="33.02" y="152.4" size="1.778" layer="95"/>
-<pinref part="UART" gate="-2" pin="S"/>
+<pinref part="SV4" gate="G$1" pin="2"/>
+<wire x1="38.1" y1="152.4" x2="30.48" y2="152.4" width="0.1524" layer="91"/>
 </segment>
 </net>
@@
 </segment>
 <segment>
+<label x="33.02" y="149.86" size="1.778" layer="95"/>
+<pinref part="SV4" gate="G$1" pin="3"/>
 <wire x1="30.48" y1="149.86" x2="38.1" y2="149.86" width="0.1524" layer="91"/>
-<label x="33.02" y="149.86" size="1.778" layer="95"/>
-<pinref part="UART" gate="-3" pin="S"/>
 </segment>
 </net>
@@
 </segment>
 <segment>
-<pinref part="I2C" gate="-1" pin="S"/>
-<wire x1="57.15" y1="78.74" x2="64.77" y2="78.74" width="0.1524" layer="91"/>
-<label x="64.77" y="78.486" size="1.778" layer="95" rot="R180"/>
+<label x="56.642" y="58.674" size="1.778" layer="95"/>
+<pinref part="SV3" gate="1" pin="1"/>
+<wire x1="60.96" y1="58.42" x2="55.88" y2="58.42" width="0.1524" layer="91"/>
 </segment>
 </net>
@@
 </segment>
 <segment>
-<pinref part="I2C" gate="-2" pin="S"/>
-<wire x1="57.15" y1="81.28" x2="64.77" y2="81.28" width="0.1524" layer="91"/>
-<label x="64.77" y="81.026" size="1.778" layer="95" rot="R180"/>
-</segment>
-</net>
+<label x="37.846" y="58.674" size="1.778" layer="95" rot="MR0"/>
+<pinref part="SV3" gate="1" pin="2"/>
+<wire x1="33.02" y1="58.42" x2="40.64" y2="58.42" width="0.1524" layer="91"/>
+</segment>
+</net>

Commit message: trinocular: rpicam_v3 + gerbers
Parts:
- removed SV3: (no value), con-lstb:MA03-2
- added SV5: (no value), con-lstb:MA20-2
- added X3: (no value), con-ptr500:AK500/2
Connections:
- net +5V: now also SV5.2, SV5.4, X3-1.KL; no longer SV3.4
- net GND: now also SV5.14, SV5.25, SV5.30, SV5.34, SV5.39, SV5.6, SV5.9, X3-2.KL; no longer SV3.3
- net SCL: now also SV5.5; no longer SV3.2
- net SDA: now also SV5.3; no longer SV3.1
Other:
- note removed: "TODO: - light sensor conn. - LED ctrl. connectors (2) - camera hole"
- moved on the sheet: ISP-1, ISP-2, ISP-3, ISP-4, ISP-5, ISP-6, ISP-7, ISP-8
